File: Projeto_exemplo_2025-1/Projeto_exemplo_2025-1.kicad_sch (KiCad schematic)
At the start: 15 parts, among them J1 Conn_01x02, U1 LM317

Commit message: Add files via upload
Parts:
- C1: footprint (none) -> Capacitor_THT:C_Disc_D6.0mm_W2.5mm_P5.00mm
- C2: footprint (none) -> Capacitor_THT:CP_Radial_D5.0mm_P2.50mm
- D2, D3, D4, D5: footprint (none) -> LED_THT:LED_D5.0mm
- R1, R2, R3, R4, R5: footprint (none) -> Resistor_THT:R_Axial_DIN0207_L6.3mm_D2.5mm_P10.16mm_Horizontal
Changed lines of the file:
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@@
       (effects (font (size 1.27 1.27)) (justify right) hide)
     )
-    (property "Footprint" "" (at 135.89 101.6 0)
+    (property "Footprint" "LED_THT:LED_D5.0mm" (at 135.89 101.6 0)
       (effects (font (size 1.27 1.27)) hide)
     )
@@
       (effects (font (size 1.27 1.27)) (justify right) hide)
     )
-    (property "Footprint" "" (at 146.05 101.6 0)
+    (property "Footprint" "LED_THT:LED_D5.0mm" (at 146.05 101.6 0)
       (effects (font (size 1.27 1.27)) hide)
     )
@@
       (effects (font (size 1.27 1.27)) (justify right) hide)
     )
-    (property "Footprint" "" (at 125.73 101.6 0)
+    (property "Footprint" "LED_THT:LED_D5.0mm" (at 125.73 101.6 0)
       (effects (font (size 1.27 1.27)) hide)
     )
@@
       (effects (font (size 1.27 1.27)) (justify left))
     )
-    (property "Footprint" "" (at 115.2652 102.87 0)
+    (property "Footprint" "Capacitor_THT:C_Disc_D6.0mm_W2.5mm_P5.00mm" (at 115.2652 102.87 0)
       (effects (font (size 1.27 1.27)) hide)
     )
@@
       (effects (font (size 1.27 1.27)) (justify left))
     )
-    (property "Footprint" "" (at 154.432 90.17 90)
+    (property "Footprint" "Resistor_THT:R_Axial_DIN0207_L6.3mm_D2.5mm_P10.16mm_Horizontal" (at 154.432 90.17 90)
       (effects (font (size 1.27 1.27)) hide)
     )
@@
       (effects (font (size 1.27 1.27)) (justify left))
     )
-    (property "Footprint" "" (at 123.952 90.17 90)
+    (property "Footprint" "Resistor_THT:R_Axial_DIN0207_L6.3mm_D2.5mm_P10.16mm_Horizontal" (at 123.952 90.17 90)
       (effects (font (size 1.27 1.27)) hide)
     )
@@
       (effects (font (size 1.27 1.27)) (justify left))
     )
-    (property "Footprint" "" (at 93.472 97.79 90)
+    (property "Footprint" "Resistor_THT:R_Axial_DIN0207_L6.3mm_D2.5mm_P10.16mm_Horizontal" (at 93.472 97.79 90)
       (effects (font (size 1.27 1.27)) hide)
     )
@@
       (effects (font (size 1.27 1.27)) (justify right) hide)
     )
-    (property "Footprint" "" (at 156.21 101.6 0)
+    (property "Footprint" "LED_THT:LED_D5.0mm" (at 156.21 101.6 0)
       (effects (font (size 1.27 1.27)) hide)
     )
@@
       (effects (font (size 1.27 1.27)) (justify left))
     )
-    (property "Footprint" "" (at 134.112 90.17 90)
+    (property "Footprint" "Resistor_THT:R_Axial_DIN0207_L6.3mm_D2.5mm_P10.16mm_Horizontal" (at 134.112 90.17 90)
       (effects (font (size 1.27 1.27)) hide)
     )
@@
       (effects (font (size 1.27 1.27)) (justify left))
     )
-    (property "Footprint" "" (at 144.272 90.17 90)
+    (property "Footprint" "Resistor_THT:R_Axial_DIN0207_L6.3mm_D2.5mm_P10.16mm_Horizontal" (at 144.272 90.17 90)
       (effects (font (size 1.27 1.27)) hide)
     )
@@
       (effects (font (size 1.27 1.27)) (justify left))
     )
-    (property "Footprint" "" (at 107.6452 102.87 0)
-      (effects (font (size 1.27 1.27)) hide)
-    )
+    (property "Footprint" "Capacitor_THT:CP_Radial_D5.0mm_P2.50mm" (at 107.6452 102.87 0)
+      (effects (font (size 1.27 1.27)) hide)
+    )

Commit message: yjrhyyrssjyyrsyjjnyg
Parts:
- J1: footprint (none) -> Projeto_exemplo_2025-1:KRE
Changed lines of the file:
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@@
       (effects (font (size 1.27 1.27)))
     )
-    (property "Footprint" "" (at 64.77 92.71 0)
+    (property "Footprint" "Projeto_exemplo_2025-1:KRE" (at 64.77 92.71 0)
       (effects (font (size 1.27 1.27)) hide)
     )

Commit message: anderson gostoso
Parts:
- RV1: footprint (none) -> Potentiometer_THT:Potentiometer_Piher_T-16H_Single_Horizontal
Changed lines of the file:
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@@
       (effects (font (size 1.27 1.27)) (justify right))
     )
-    (property "Footprint" "" (at 86.36 106.68 0)
+    (property "Footprint" "Potentiometer_THT:Potentiometer_Piher_T-16H_Single_Horizontal" (at 86.36 106.68 0)
       (effects (font (size 1.27 1.27)) hide)
     )
