File: Projeto_exemplo_ifsc_2025.1/Projeto_exemplo_ifsc_2025.1.kicad_pcb (KiCad board)
At the start: 2 copper layers, 45.5 x 36 mm, 15 parts, among them J1 Conn_01x02, U2 LM317_TO-220

Commit message: arfhmk
Parts:
- moved D4 2.21 mm to (233.8, 135.2)
- moved R4 2.21 mm to (243.3, 135.2)
- moved R3 1.20 mm to (243.3, 142.7)
- moved D3 1.20 mm to (233.6, 142.7)
- moved R2 0.53 mm to (243.4, 150.0)
- moved D2 0.53 mm to (233.7, 150.0)
Connections:
- RV1 pad 1: Net-(U2-ADJ) -> GNDREF
- RV1 pad 3: GNDREF -> Net-(U2-ADJ)
Routing:
- net Net-(U2-VO): track 72.8 -> 70.8 mm
Changed lines of the file:
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@@
 	(footprint "aaProprio:Led_5mm"
 		(layer "F.Cu")
-		(at 233.9 133)
+		(at 233.81 135.21)
 		(property "Reference" "D4"
 			(at 0 -4 0)
@@
 	(footprint "aaProprio:Resistor_330_1_4W"
 		(layer "F.Cu")
-		(at 243.4 133 180)
+		(at 243.31 135.21 180)
 		(property "Reference" "R4"
 			(at 0 -2 0)
@@
 	(footprint "aaProprio:Led_5mm"
 		(layer "F.Cu")
-		(at 233.7 149.5)
+		(at 233.69 150.03)
 		(property "Reference" "D2"
 			(at 0 -3.5 0)
@@
 			(layers "*.Cu" "*.Mask")
 			(remove_unused_layers no)
-			(net 9 "Net-(U2-ADJ)")
+			(net 2 "GNDREF")
 			(pinfunction "1")
 			(pintype "passive")
@@
 			(layers "*.Cu" "*.Mask")
 			(remove_unused_layers no)
-			(net 2 "GNDREF")
+			(net 9 "Net-(U2-ADJ)")
 			(pinfunction "3")
 			(pintype "passive")
@@
 	(footprint "aaProprio:Resistor_330_1_4W"
 		(layer "F.Cu")
-		(at 243.4 141.5 180)
+		(at 243.31 142.7 180)
 		(property "Reference" "R3"
 			(at 0 -2 0)
@@
 	(footprint "aaProprio:Led_5mm"
 		(layer "F.Cu")
-		(at 233.7 141.5)
+		(at 233.61 142.7)
 		(property "Reference" "D3"
 			(at 0 -3.5 0)
@@
 	(footprint "aaProprio:Resistor_330_1_4W"
 		(layer "F.Cu")
-		(at 243.4 149.5 180)
+		(at 243.39 150.03 180)
 		(property "Reference" "R2"
 			(at 0 -2 0)
@@
 	)
 	(gr_text_box "Projeto exemplo (Luminaria)\nFelipe S Kraemer"
-		(start 232.65 126.75)
-		(end 249.15 129.25)
+		(start 232.65 128)
+		(end 249.15 130.5)
 		(margins 1.0025 1.0025 1.0025 1.0025)
 		(layer "B.Cu")
@@
 	)
 	(gr_text_box "Projeto exemplo (Luminaria)\nFelipe S Kraemer"
-		(start 232.65 126.75)
-		(end 249.15 129.25)
+		(start 232.65 128)
+		(end 249.15 130.5)
 		(margins 1.0025 1.0025 1.0025 1.0025)
 		(layer "F.SilkS")
@@
 	)
 	(segment
-		(start 248.4 141.5)
-		(end 248.4 149.5)
-		(width 1.016)
+		(start 244.37 131.27)
+		(end 228.13 131.27)
+		(width 1)
 		(layer "B.Cu")
 		(net 1)
@@
 	)
 	(segment
-		(start 228.9 130.5)
-		(end 245.9 130.5)
-		(width 1.016)
+		(start 228.13 131.27)
+		(end 222.4 137)
+		(width 1)
 		(layer "B.Cu")
 		(net 1)
 	)
 	(segment
-		(start 248.4 133)
-		(end 248.4 141.5)
-		(width 1.016)
-		(layer "B.Cu")
-		(net 1)
-	)
-	(segment
-		(start 222.4 137)
-		(end 228.9 130.5)
-		(width 1.016)
+		(start 248.39 150.03)
+		(end 248.39 157.99)
+		(width 1)
 		(layer "B.Cu")
 		(net 1)
@@
 	)
 	(segment
-		(start 245.9 130.5)
-		(end 248.4 133)
-		(width 1.016)
-		(layer "B.Cu")
-		(net 1)
-	)
-	(segment
 		(start 224.9 144)
 		(end 223.9 144)
@@
 	)
 	(segment
+		(start 248.39 157.99)
+		(end 248.4 158)
+		(width 1)
+		(layer "B.Cu")
+		(net 1)
+	)
+	(segment
+		(start 248.31 149.95)
+		(end 248.39 150.03)
+		(width 1)
+		(layer "B.Cu")
+		(net 1)
+	)
+	(segment
+		(start 248.31 135.21)
+		(end 244.37 131.27)
+		(width 1)
+		(layer "B.Cu")
+		(net 1)
+	)
+	(segment
 		(start 223.9 144)
 		(end 222.4 142.5)
@@
 	)
 	(segment
+		(start 248.31 135.21)
+		(end 248.31 142.7)
+		(width 1)
+		(layer "B.Cu")
+		(net 1)
+	)
+	(segment
 		(start 224.9 144)
 		(end 224.9 147)
@@
 	)
 	(segment
-		(start 248.4 149.5)
-		(end 248.4 158)
-		(width 1.016)
+		(start 248.31 142.7)
+		(end 248.31 149.95)
+		(width 1)
 		(layer "B.Cu")
 		(net 1)
@@
 	)
 	(segment
-		(start 234.9 149.5)
-		(end 238.4 149.5)
-		(width 1.016)
+		(start 238.39 150.03)
+		(end 234.89 150.03)
+		(width 1)
 		(layer "B.Cu")
 		(net 4)
 	)
 	(segment
-		(start 238.4 141.5)
-		(end 234.9 141.5)
-		(width 1.016)
+		(start 234.81 142.7)
+		(end 238.31 142.7)
+		(width 1)
 		(layer "B.Cu")
 		(net 5)
 	)
 	(segment
-		(start 235.1 133)
-		(end 238.4 133)
-		(width 1.016)
+		(start 238.31 135.21)
+		(end 235.01 135.21)
+		(width 1)
 		(layer "B.Cu")
 		(net 6)
@@
 	)
 	(segment
-		(start 216.4 144.5)
-		(end 212.3 144.5)
+		(start 212.3 149.5)
+		(end 212.3 154.5)
 		(width 1.016)
 		(layer "B.Cu")
-		(net 9)
-	)
-	(segment
-		(start 216.9 145)
-		(end 216.4 144.5)
-		(width 1.016)
-		(layer "B.Cu")
